Commit message: still debugging convex hull bullet collision checking

File: cdcpd/fake_robot.urdf (robot description, URDF)
Before this commit: robot fake_robot, 1 links, 0 joints
Links:
- removed link fake_robot_link
- added link mock_camera_link; visual cylinder length=0.05 radius=0.02; visual sphere radius=0.02
